File: hardware/recorder.kicad_pcb (KiCad board)
At the start: 2 copper layers, 105 x 85 mm, 30 parts, among them J1 Nano TX V2, J2 Buck MP1584E, J3 LiPo 3S / PSU, J4 USB-Serial, SW1 SW_Push, SW2 SW_Push, SW3 SW_SPST, U1 Raspberry Pi Pico

Commit message: Fit the real MP1584EN buck module: custom footprint and re-layout
The module arrived, so J2 is no longer a placeholder header. Derived
its footprint from the product photos by measuring the pad positions
in the image rather than eyeballing them: eight holes in four pairs,
board 22.3x16.8mm, columns at +/-9.45mm and rows at +/-6.70/4.16mm
with the expected 2.54mm pair pitch, symmetric about the centre.

Pin orientation comes from both photos agreeing: the underside silk
reads OUT-/IN- over OUT+/IN+, which mirrors to IN on the left and OUT
on the right seen from the component side, matching the board's own
+/- marks sitting on the output end.

Moving to a 22.3mm-wide part meant re-placing J2 (it would have sat on
top of the Pico at the old position) and rerouting VBAT and +5V. The
module now sits bottom-right, clear of both the Pico and the corner
mounting hole, whose courtyard is a 3.45mm circle and caught the first
two attempts.

Still DRC clean: 0 violations, 0 unconnected, ERC 0/0, Gerbers export.

The dimensions come from image analysis, not calipers, so README now
says to check the eight holes against a 1:1 printout before ordering
and which two constants to edit if they are off.

Co-Authored-By: Claude Opus 5 <noreply@anthropic.com>
Parts:
- removed the H1 at (14.0, 14.0)
- added H4: , MountingHole_3.2mm_M3, F.Cu at (111.0, 91.0)
- J2: footprint PinHeader_1x04_P2.54mm_Vertical -> MP1584EN_Module
- moved H2 123.8 mm to (111.0, 14.0)
- moved H1 97.0 mm to (14.0, 14.0)
- moved H3 97.0 mm to (14.0, 91.0)
- moved J2 4.00 mm to (96.0, 80.0)
- renumbered H2 to H1, H3 to H2, H4 to H3
Routing:
- net +5V: track 88.3 -> 103.1 mm
- net GND: track 13.0 -> 18.1 mm
Other:
- board text removed: "BUCK 5V"
